Commit message: fix: gimli prototype args

File: nav2_bringup/bringup/urdf/turtlebot3_waffle.urdf (robot description, URDF)
Before this commit: robot turtlebot3_waffle, 13 links, 12 joints
Links:
- link wheel_left_link: geometry collision cylinder length=0.018 radius=0.8; visual mesh filename=package://turtlebot3_gazebo/models/turtlebot3_common/meshes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 scale=0.001 0.001 0.001
- link wheel_right_link: geometry collision cylinder length=0.018 radius=0.8; visual mesh filename=package://turtlebot3_gazebo/models/turtlebot3_common/meshes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 scale=0.001 0.001 0.001
Joints:
- joint wheel_left_joint: origin xyz=0.0 0.144 0.023 rpy=-1.57 0 0 -> xyz=0.0 0.5 0.023 rpy=-1.57 0 0
- joint wheel_right_joint: origin xyz=0.0 -0.144 0.023 rpy=-1.57 0 0 -> xyz=0.0 -0.5 0.023 rpy=-1.57 0 0

Commit message: fix: lidar

File: nav2_bringup/bringup/urdf/turtlebot3_waffle.urdf (robot description, URDF)
Before this commit: robot turtlebot3_waffle, 13 links, 12 joints
Joints:
- joint scan_joint: origin xyz=-0.064 0 0.122 rpy=0 0 0 -> xyz=-0.52 0 0.122 rpy=3.14159 0 0

Commit message: fix: updates

File: nav2_bringup/bringup/urdf/turtlebot3_waffle.urdf (robot description, URDF)
Before this commit: robot turtlebot3_waffle, 13 links, 12 joints
Joints:
- joint scan_joint: origin xyz=-0.52 0 0.122 rpy=3.14159 0 0 -> xyz=-0.52 0 0.0 rpy=0.0 0.0 0
